Commit message: Updated

File: src/RobotModels/ALOHA_MED/robot.urdf (robot description, URDF)
Before this commit: robot ALOHA_MED, 7 links, 6 joints
Joints:
- removed joint joint_6_wrist_3
- added joint : type revolute, parent link_5_aloha_lc_v1_4, child fcg_eef_aloha_lc_v1_4, origin xyz=0.060333 -0.00143286 -0.018425 rpy=-1.5708 1.62394e-05 1.54705, axis 0 0 1, limit lower=-1.5708 upper=1.5708 effort=10 velocity=10
- joint joint_2_shoulder_lift: limit lower=-3.141592653589793 upper=3.141592653589793 effort=10 velocity=10 -> lower=0 upper=3.14159 effort=10 velocity=10
- joint joint_3_elbow: limit lower=-3.141592653589793 upper=3.141592653589793 effort=10 velocity=10 -> lower=0 upper=3.14159 effort=10 velocity=10
- joint joint_4_wrist_1: limit lower=-3.141592653589793 upper=3.141592653589793 effort=10 velocity=10 -> lower=-1.5708 upper=1.5708 effort=10 velocity=10; origin xyz=0.0878508 -0.0014563 -0.0385968 rpy=-1.5708 0.0251682 1.55422 -> xyz=0.0878508 -0.0014563 -0.0385968 rpy=-1.5708 -7e-12 1.55422
- joint joint_5_wrist_2: limit lower=-3.141592653589793 upper=3.141592653589793 effort=10 velocity=10 -> lower=-1.5708 upper=1.5708 effort=10 velocity=10; origin xyz=-4.60594e-07 -0.0198 -0.07496 rpy=1.5708 1.53515 -2.32623e-05 -> xyz=-4.60594e-07 -0.0198 -0.07496 rpy=1.5708 1.55422 -2.32623e-05
